Commit message: modified rviz.launch.py for SO-100 arm simulation

File: urdf/so_100_arm.urdf (robot description, URDF)
Before this commit: robot so_100_arm, 8 links, 7 joints
Joints:
- joint Elbow: limit (none) -> lower=0 upper=3.1415926535 effort=100 velocity=1.0
- joint Gripper: limit (none) -> lower=0 upper=1.5707963268 effort=50 velocity=0.5
- joint Shoulder_Pitch: limit (none) -> lower=0 upper=3.1415926535 effort=100 velocity=1.0
- joint Shoulder_Rotation: limit (none) -> lower=0 upper=3.1415926535 effort=100 velocity=1.0
- joint Wrist_Pitch: limit (none) -> lower=-1.5707963268 upper=1.5707963268 effort=100 velocity=1.0
- joint Wrist_Roll: limit (none) -> lower=-1.5707963268 upper=1.5707963268 effort=100 velocity=1.0

File: urdf/so_100_arm_5dof_hardware.urdf (robot description, URDF)
Before this commit: robot so_100_arm, 8 links, 7 joints
Joints:
- joint Elbow: limit (none) -> lower=0.0 upper=3.14159 effort=100 velocity=1.0
- joint Gripper: limit (none) -> lower=0.0 upper=1.570796 effort=50 velocity=0.5
- joint Shoulder_Pitch: limit (none) -> lower=0.0 upper=3.14159 effort=100 velocity=1.0
- joint Shoulder_Rotation: limit (none) -> lower=0.0 upper=3.14159 effort=100 velocity=1.0
- joint Wrist_Pitch: limit (none) -> lower=-1.570796 upper=1.570796 effort=100 velocity=1.0
- joint Wrist_Roll: limit (none) -> lower=-1.570796 upper=1.570796 effort=100 velocity=1.0
